File: KiCad PiHat/Lec18-PCB_kicad.kicad_sch (KiCad schematic)
At the start: 6 parts

Commit message: Ongoing work
Continued work on schematic and PCB
Parts:
- added J1, J2, J3: (no value), symbol Connector_Generic:Conn_01x03
- added J4, J5, J6, J7: (no value), symbol Connector_Generic:Conn_01x04
- added J8, J9: (no value), symbol Connector:Screw_Terminal_01x02
- added R1, R2, R3: (no value), symbol Device:R
- A1: footprint (none) -> Module:Arduino_Nano; symbol MCU_Module:Arduino_Nano_v2.x -> MCU_Module:Arduino_Nano_Every
- MK1, MK2, MK3, MK4: value (none) -> M2.5; footprint (none) -> MountingHole:MountingHole_2.7mm_M2.5
- P1: value (none) -> Conn_02x20_Odd_Even; footprint (none) -> Connector_PinSocket_2.54mm:PinSocket_2x20_P2.54mm_Vertical
Connections:
- net +5V: now also A1.30 (VIN), J1.2 (Pin_2), J2.2 (Pin_2), J3.2 (Pin_2), J6.4 (Pin_4), J7.4 (Pin_4), J8.2 (Pin_2), J9.2 (Pin_2); no longer P1.2 (Pin_2), P1.4 (Pin_4)
- net GND: now also A1.29 (GND), A1.4 (GND), J1.1 (Pin_1), J2.1 (Pin_1), J3.1 (Pin_1), J6.1 (Pin_1), J7.1 (Pin_1), J8.1 (Pin_1), J9.1 (Pin_1), R2.2
- net +3V3: no longer names the net of P1.1 (Pin_1), P1.17 (Pin_17)
- net GPIO15(RXD0) renamed GPIO14(TXD0_5V)
- net GPIO14(TXD0_5V): now also R1.1; no longer P1.10 (Pin_10)
- new net: P1.2 (Pin_2), P1.4 (Pin_4)
- new net: R2.1, R3.2
- new net GPIO15(RXD0_3.3V): P1.10 (Pin_10), R1.2, R3.1
- new net IN1(MOTOR_LEFT): J4.1 (Pin_1)
- new net IN1(MOTOR_RIGHT): J5.1 (Pin_1)
- new net IN2(MOTOR_LEFT): J4.2 (Pin_2)
- new net IN2(MOTOR_RIGHT): J5.2 (Pin_2)
- new net IN3(MOTOR_LEFT): J4.3 (Pin_3)
- new net IN3(MOTOR_RIGHT): J5.3 (Pin_3)
- new net IN4(MOTOR_LEFT): J4.4 (Pin_4)
- new net IN4(MOTOR_RIGHT): J5.4 (Pin_4)
Other:
- moved on the sheet: P1

Commit message: Finished Schematic
Schematic finished. Sanity check and routing coming next
Parts:
- added J10: (no value), symbol Connector:USB_C_Receptacle_USB2.0
- added R4, R5, R6: (no value), symbol Device:R
- A1: footprint Module:Arduino_Nano -> (none); symbol MCU_Module:Arduino_Nano_Every -> Teensy:Teensy4.0
- P1: value Conn_02x20_Odd_Even -> (none); footprint Connector_PinSocket_2.54mm:PinSocket_2x20_P2.54mm_Vertical -> (none)
Connections:
- net +5V: now also A1.33 (VIN), J8.1 (Pin_1), J9.1 (Pin_1), J10.A4 (VBUS), J10.A9 (VBUS), J10.B4 (VBUS), J10.B9 (VBUS); no longer A1.30 (VIN), J8.2 (Pin_2), J9.2 (Pin_2)
- net GND: now also A1.1 (GND), A1.17 (GND), A1.32 (GND), A1.47 (GND), J8.2 (Pin_2), J9.2 (Pin_2), R3.2, J10.A1 (GND), J10.A12 (GND), J10.B1 (GND), J10.B12 (GND), J10.S1 (SHIELD), R6.2; no longer A1.29 (GND), A1.4 (GND), J8.1 (Pin_1), J9.1 (Pin_1), R2.2
- net GPIO17(GEN0): now also J3.3 (Pin_3)
- net GPIO22(GEN3): now also J2.3 (Pin_3)
- net GPIO5: now also J1.3 (Pin_3)
- net IN1(MOTOR_LEFT): now also A1.11 (9_OUT1C)
- net IN1(MOTOR_RIGHT): now also A1.4 (2_OUT2)
- net IN2(MOTOR_LEFT): now also A1.10 (8_TX2_IN1)
- net IN2(MOTOR_RIGHT): now also A1.5 (3_LRCLK2)
- net IN3(MOTOR_LEFT): now also A1.9 (7_RX2_OUT1A)
- net IN3(MOTOR_RIGHT): now also A1.6 (4_BCLK2)
- net IN4(MOTOR_LEFT): now also A1.8 (6_OUT1D)
- net IN4(MOTOR_RIGHT): now also A1.7 (5_IN2)
- net Ultrasonic_Front_Echo: now reaches R2.1
- net Ultrasonic_Front_Echo: now also A1.26 (19_A5_SCL0), R1.2; no longer R3.2
- net at J6.2 (Pin_2): now also R1.1
- net Ultrasonic_Front_Trig: now reaches J6.3 (Pin_3)
- net Ultrasonic_Front_Trig: now also A1.25 (18_A4_SDA0)
- net Teensy_to_PI: now reaches A1.3 (1_TX1_CTX2_MISO1)
- net Teensy_to_PI: now also P1.10 (Pin_10)
- net at J7.2 (Pin_2): now also R4.1
- net Ultrasonic_Left_Trig: now reaches J7.3 (Pin_3)
- net Ultrasonic_Left_Trig: now also A1.29 (22_A8_CTX1)
- net GPIO14(TXD0) renamed PI_to_Teensy
- removed net GPIO14(TXD0_5V): A1.1 (TX1), R1.1
- removed net GPIO15(RXD0_3.3V): P1.10 (Pin_10), R1.2, R3.1
- new net: R5.2, R6.1
- new net: R2.2, R3.1
- new net Ultrasonic_Left_Echo: A1.30 (23_A9_CRX1_MCLK1), R4.2, R5.1
Other:
- moved on the sheet: J1, J2, J3, J4, J5, J6, J7, J8, J9

Commit message: routing complete
Parts:
- J10: symbol Connector:USB_C_Receptacle_USB2.0 -> Connector:USB_C_Receptacle
Changed lines of the file:
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@@
     (pin "1")
   )
-  (symbol (lib_id "power:GND") (at 43.18 135.89 0) (unit 1)
-    (in_bom yes) (on_board yes)
-    (property "Reference" "#PWR0114" (id 0) (at 43.18 142.24 0)
-      (effects (font (size 1.27 1.27)) hide)
-    )
-    (property "Value" "GND" (id 1) (at 43.18 139.7 0))
-    (property "Footprint" "" (id 2) (at 43.18 135.89 0))
-    (property "Datasheet" "" (id 3) (at 43.18 135.89 0))
+  (symbol (lib_id "power:GND") (at 34.29 153.67 0) (unit 1)
+    (in_bom yes) (on_board yes)
+    (property "Reference" "#PWR0114" (id 0) (at 34.29 160.02 0)
+      (effects (font (size 1.27 1.27)) hide)
+    )
+    (property "Value" "GND" (id 1) (at 34.29 157.48 0))
+    (property "Footprint" "" (id 2) (at 34.29 153.67 0))
+    (property "Datasheet" "" (id 3) (at 34.29 153.67 0))
     (pin "1")
   )
@@
     (pin "1")
   )
-  (symbol (lib_id "power:GND") (at 35.56 135.89 0) (unit 1)
-    (in_bom yes) (on_board yes)
-    (property "Reference" "#PWR0115" (id 0) (at 35.56 142.24 0)
-      (effects (font (size 1.27 1.27)) hide)
-    )
-    (property "Value" "GND" (id 1) (at 35.56 139.7 0))
-    (property "Footprint" "" (id 2) (at 35.56 135.89 0))
-    (property "Datasheet" "" (id 3) (at 35.56 135.89 0))
+  (symbol (lib_id "power:GND") (at 26.67 153.67 0) (unit 1)
+    (in_bom yes) (on_board yes)
+    (property "Reference" "#PWR0115" (id 0) (at 26.67 160.02 0)
+      (effects (font (size 1.27 1.27)) hide)
+    )
+    (property "Value" "GND" (id 1) (at 26.67 157.48 0))
+    (property "Footprint" "" (id 2) (at 26.67 153.67 0))
+    (property "Datasheet" "" (id 3) (at 26.67 153.67 0))
     (pin "1")
   )
@@
     (pin "2")
   )
-  (symbol (lib_id "power:+5V") (at 58.42 97.79 0) (unit 1)
-    (in_bom yes) (on_board yes)
-    (property "Reference" "#PWR0113" (id 0) (at 58.42 101.6 0)
-      (effects (font (size 1.27 1.27)) hide)
-    )
-    (property "Value" "+5V" (id 1) (at 58.42 94.234 0))
-    (property "Footprint" "" (id 2) (at 58.42 97.79 0))
-    (property "Datasheet" "" (id 3) (at 58.42 97.79 0))
+  (symbol (lib_id "power:+5V") (at 49.53 87.63 0) (unit 1)
+    (in_bom yes) (on_board yes)
+    (property "Reference" "#PWR0113" (id 0) (at 49.53 91.44 0)
+      (effects (font (size 1.27 1.27)) hide)
+    )
+    (property "Value" "+5V" (id 1) (at 49.53 84.074 0))
+    (property "Footprint" "" (id 2) (at 49.53 87.63 0))
+    (property "Datasheet" "" (id 3) (at 49.53 87.63 0))
     (pin "1")
   )
@@
     (pin "1")
   )
-  (symbol (lib_id "Connector:USB_C_Receptacle_USB2.0") (at 43.18 113.03 0) (unit 1)
-    (in_bom yes) (on_board yes) (fields_autoplaced)
-    (property "Reference" "J10" (id 0) (at 43.18 90.17 0))
-    (property "Value" "" (id 1) (at 43.18 92.71 0))
-    (property "Footprint" "" (id 2) (at 46.99 113.03 0)
-      (effects (font (size 1.27 1.27)) hide)
-    )
-    (property "Datasheet" "https://www.usb.org/sites/default/files/documents/usb_type-c.zip" (id 3) (at 46.99 113.03 0)
+  (symbol (lib_id "Connector:USB_C_Receptacle") (at 34.29 113.03 0) (unit 1)
+    (in_bom yes) (on_board yes)
+    (property "Reference" "J10" (id 0) (at 34.29 90.17 0))
+    (property "Value" "" (id 1) (at 29.21 82.55 0))
+    (property "Footprint" "" (id 2) (at 38.1 113.03 0)
+      (effects (font (size 1.27 1.27)) hide)
+    )
+    (property "Datasheet" "https://www.usb.org/sites/default/files/documents/usb_type-c.zip" (id 3) (at 38.1 113.03 0)
       (effects (font (size 1.27 1.27)) hide)
     )
     (pin "A1")
+    (pin "A10")
+    (pin "A11")
     (pin "A12")
+    (pin "A2")
+    (pin "A3")
     (pin "A4")
     (pin "A5")
@@
     (pin "A9")
     (pin "B1")
+    (pin "B10")
+    (pin "B11")
     (pin "B12")
+    (pin "B2")
+    (pin "B3")
     (pin "B4")
     (pin "B5")

Commit message: not sure tbh
Parts:
- A1: value (none) -> Teensy_4.0; footprint (none) -> teensy:Teensy40
- J1: value (none) -> Servo_BEEG; footprint (none) -> Connector_PinSocket_2.54mm:PinSocket_1x03_P2.54mm_Vertical
- J10: value (none) -> USB_C_Receptacle_USB2.0; footprint (none) -> Connector_USB:USB_C_Receptacle_GCT_USB4085
- J2: value (none) -> Servo_SHOOT; footprint (none) -> Connector_PinSocket_2.54mm:PinSocket_1x03_P2.54mm_Vertical
- J3: value (none) -> Servo_EXTRA; footprint (none) -> Connector_PinSocket_2.54mm:PinSocket_1x03_P2.54mm_Vertical
- J4: value (none) -> Motor_Driver_Left; footprint (none) -> Connector_PinSocket_2.54mm:PinSocket_1x04_P2.54mm_Vertical
- J5: value (none) -> Motor_Driver_Right; footprint (none) -> Connector_PinSocket_2.54mm:PinSocket_1x04_P2.54mm_Vertical
- J6: value (none) -> Ultrasonic_Front; footprint (none) -> Connector_PinSocket_2.54mm:PinSocket_1x04_P2.54mm_Vertical
- J7: value (none) -> Ultrasonic_Left; footprint (none) -> Connector_PinSocket_2.54mm:PinSocket_1x04_P2.54mm_Vertical
- J8: value (none) -> Motor_Power_Left; footprint (none) -> TerminalBlock:TerminalBlock_bornier-2_P5.08mm
- J9: value (none) -> Motor_Power_Right; footprint (none) -> TerminalBlock:TerminalBlock_bornier-2_P5.08mm
- P1: value (none) -> RaspberryPi_Connector; footprint (none) -> Connector_PinSocket_2.54mm:PinSocket_2x20_P2.54mm_Vertical
- R1, R2, R3, R4, R5, R6: value (none) -> 1k; footprint (none) -> Resistor_THT:R_Axial_DIN0207_L6.3mm_D2.5mm_P7.62mm_Horizontal
Changed lines of the file:
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@@
       (effects (font (size 1.27 1.27)) hide)
     )
-    (property "Value" "" (id 1) (at 198.12 98.044 0))
+    (property "Value" "+5V" (id 1) (at 198.12 98.044 0))
     (property "Footprint" "" (id 2) (at 198.12 101.6 0))
     (property "Datasheet" "" (id 3) (at 198.12 101.6 0))
@@
     (in_bom yes) (on_board yes)
     (property "Reference" "P1" (id 0) (at 67.31 24.9682 0))
-    (property "Value" "" (id 1) (at 67.31 27.2796 0))
-    (property "Footprint" "" (id 2) (at -57.15 77.47 0)
+    (property "Value" "RaspberryPi_Connector" (id 1) (at 67.31 27.2796 0))
+    (property "Footprint" "Connector_PinSocket_2.54mm:PinSocket_2x20_P2.54mm_Vertical" (id 2) (at -57.15 77.47 0)
       (effects (font (size 1.27 1.27)) hide)
     )
@@
       (effects (font (size 1.27 1.27)) (justify left))
     )
-    (property "Value" "" (id 1) (at 129.54 167.6399 0)
-      (effects (font (size 1.27 1.27)) (justify left))
-    )
-    (property "Footprint" "" (id 2) (at 125.222 166.37 90)
+    (property "Value" "1k" (id 1) (at 129.54 167.6399 0)
+      (effects (font (size 1.27 1.27)) (justify left))
+    )
+    (property "Footprint" "Resistor_THT:R_Axial_DIN0207_L6.3mm_D2.5mm_P7.62mm_Horizontal" (id 2) (at 125.222 166.37 90)
       (effects (font (size 1.27 1.27)) hide)
     )
@@
       (effects (font (size 1.27 1.27)) (justify left))
     )
-    (property "Value" "" (id 1) (at 129.54 135.8899 0)
-      (effects (font (size 1.27 1.27)) (justify left))
-    )
-    (property "Footprint" "" (id 2) (at 125.222 134.62 90)
+    (property "Value" "1k" (id 1) (at 129.54 135.8899 0)
+      (effects (font (size 1.27 1.27)) (justify left))
+    )
+    (property "Footprint" "Resistor_THT:R_Axial_DIN0207_L6.3mm_D2.5mm_P7.62mm_Horizontal" (id 2) (at 125.222 134.62 90)
       (effects (font (size 1.27 1.27)) hide)
     )
@@
       (effects (font (size 1.27 1.27)) (justify left))
     )
-    (property "Value" "" (id 1) (at 260.35 73.6599 0)
-      (effects (font (size 1.27 1.27)) (justify left))
-    )
-    (property "Footprint" "" (id 2) (at 257.81 72.39 0)
+    (property "Value" "Servo_BEEG" (id 1) (at 260.35 73.6599 0)
+      (effects (font (size 1.27 1.27)) (justify left))
+    )
+    (property "Footprint" "Connector_PinSocket_2.54mm:PinSocket_1x03_P2.54mm_Vertical" (id 2) (at 257.81 72.39 0)
       (effects (font (size 1.27 1.27)) hide)
     )
@@
       (effects (font (size 1.27 1.27)) (justify left))
     )
-    (property "Value" "" (id 1) (at 262.89 35.5599 0)
-      (effects (font (size 1.27 1.27)) (justify left))
-    )
-    (property "Footprint" "" (id 2) (at 260.35 33.02 0)
+    (property "Value" "Motor_Driver_Right" (id 1) (at 262.89 35.5599 0)
+      (effects (font (size 1.27 1.27)) (justify left))
+    )
+    (property "Footprint" "Connector_PinSocket_2.54mm:PinSocket_1x04_P2.54mm_Vertical" (id 2) (at 260.35 33.02 0)
       (effects (font (size 1.27 1.27)) hide)
     )
@@
       (effects (font (size 1.27 1.27)) (justify left))
     )
-    (property "Value" "" (id 1) (at 260.35 82.5499 0)
-      (effects (font (size 1.27 1.27)) (justify left))
-    )
-    (property "Footprint" "" (id 2) (at 257.81 81.28 0)
+    (property "Value" "Servo_SHOOT" (id 1) (at 260.35 82.5499 0)
+      (effects (font (size 1.27 1.27)) (justify left))
+    )
+    (property "Footprint" "Connector_PinSocket_2.54mm:PinSocket_1x03_P2.54mm_Vertical" (id 2) (at 257.81 81.28 0)
       (effects (font (size 1.27 1.27)) hide)
     )
@@
       (effects (font (size 1.27 1.27)) (justify left))
     )
-    (property "Value" "" (id 1) (at 175.26 146.0499 0)
-      (effects (font (size 1.27 1.27)) (justify left))
-    )
-    (property "Footprint" "" (id 2) (at 172.72 143.51 0)
+    (property "Value" "Ultrasonic_Front" (id 1) (at 175.26 146.0499 0)
+      (effects (font (size 1.27 1.27)) (justify left))
+    )
+    (property "Footprint" "Connector_PinSocket_2.54mm:PinSocket_1x04_P2.54mm_Vertical" (id 2) (at 172.72 143.51 0)
       (effects (font (size 1.27 1.27)) hide)
     )
@@
       (effects (font (size 1.27 1.27)) (justify left))
     )
-    (property "Value" "" (id 1) (at 129.54 128.2699 0)
-      (effects (font (size 1.27 1.27)) (justify left))
-    )
-    (property "Footprint" "" (id 2) (at 125.222 127 90)
+    (property "Value" "1k" (id 1) (at 129.54 128.2699 0)
+      (effects (font (size 1.27 1.27)) (justify left))
+    )
+    (property "Footprint" "Resistor_THT:R_Axial_DIN0207_L6.3mm_D2.5mm_P7.62mm_Horizontal" (id 2) (at 125.222 127 90)
       (effects (font (size 1.27 1.27)) hide)
     )
@@
       (effects (font (size 1.27 1.27)) (justify left))
     )
-    (property "Value" "" (id 1) (at 129.54 143.5099 0)
-      (effects (font (size 1.27 1.27)) (justify left))
-    )
-    (property "Footprint" "" (id 2) (at 125.222 142.24 90)
+    (property "Value" "1k" (id 1) (at 129.54 143.5099 0)
+      (effects (font (size 1.27 1.27)) (justify left))
+    )
+    (property "Footprint" "Resistor_THT:R_Axial_DIN0207_L6.3mm_D2.5mm_P7.62mm_Horizontal" (id 2) (at 125.222 142.24 90)
       (effects (font (size 1.27 1.27)) hide)
     )
@@
       (effects (font (size 1.27 1.27)) (justify left))
     )
-    (property "Value" "" (id 1) (at 129.54 175.2599 0)
-      (effects (font (size 1.27 1.27)) (justify left))
-    )
-    (property "Footprint" "" (id 2) (at 125.222 173.99 90)
+    (property "Value" "1k" (id 1) (at 129.54 175.2599 0)
+      (effects (font (size 1.27 1.27)) (justify left))
+    )
+    (property "Footprint" "Resistor_THT:R_Axial_DIN0207_L6.3mm_D2.5mm_P7.62mm_Horizontal" (id 2) (at 125.222 173.99 90)
       (effects (font (size 1.27 1.27)) hide)
     )
@@
       (effects (font (size 1.27 1.27)) (justify left))
     )
-    (property "Value" "" (id 1) (at 234.95 48.2599 0)
-      (effects (font (size 1.27 1.27)) (justify left))
-    )
-    (property "Footprint" "" (id 2) (at 232.41 45.72 0)
+    (property "Value" "Motor_Power_Right" (id 1) (at 234.95 48.2599 0)
+      (effects (font (size 1.27 1.27)) (justify left))
+    )
+    (property "Footprint" "TerminalBlock:TerminalBlock_bornier-2_P5.08mm" (id 2) (at 232.41 45.72 0)
       (effects (font (size 1.27 1.27)) hide)
     )
@@
       (effects (font (size 1.27 1.27)) (justify left))
     )
-    (property "Value" "" (id 1) (at 168.91 106.68 0)
-      (effects (font (size 1.27 1.27)) (justify left))
-    )
-    (property "Footprint" "" (id 2) (at 157.48 74.93 0)
+    (property "Value" "Teensy_4.0" (id 1) (at 168.91 106.68 0)
+      (effects (font (size 1.27 1.27)) (justify left))
+    )
+    (property "Footprint" "teensy:Teensy40" (id 2) (at 157.48 74.93 0)
       (effects (font (size 1.27 1.27)) hide)
     )
@@
       (effects (font (size 1.27 1.27)) (justify left))
     )
-    (property "Value" "" (id 1) (at 175.26 157.4799 0)
-      (effects (font (size 1.27 1.27)) (justify left))
-    )
-    (property "Footprint" "" (id 2) (at 172.72 154.94 0)
+    (property "Value" "Ultrasonic_Left" (id 1) (at 175.26 157.4799 0)
+      (effects (font (size 1.27 1.27)) (justify left))
+    )
+    (property "Footprint" "Connector_PinSocket_2.54mm:PinSocket_1x04_P2.54mm_Vertical" (id 2) (at 172.72 154.94 0)
       (effects (font (size 1.27 1.27)) hide)
     )
@@
       (effects (font (size 1.27 1.27)) (justify left))
     )
-    (property "Value" "" (id 1) (at 262.89 48.2599 0)
-      (effects (font (size 1.27 1.27)) (justify left))
-    )
-    (property "Footprint" "" (id 2) (at 260.35 45.72 0)
+    (property "Value" "Motor_Power_Left" (id 1) (at 262.89 48.2599 0)
+      (effects (font (size 1.27 1.27)) (justify left))
+    )
+    (property "Footprint" "TerminalBlock:TerminalBlock_bornier-2_P5.08mm" (id 2) (at 260.35 45.72 0)
       (effects (font (size 1.27 1.27)) hide)
     )
@@
       (effects (font (size 1.27 1.27)) (justify left))
     )
-    (property "Value" "" (id 1) (at 129.54 160.0199 0)
-      (effects (font (size 1.27 1.27)) (justify left))
-    )
-    (property "Footprint" "" (id 2) (at 125.222 158.75 90)
+    (property "Value" "1k" (id 1) (at 129.54 160.0199 0)
+      (effects (font (size 1.27 1.27)) (justify left))
+    )
+    (property "Footprint" "Resistor_THT:R_Axial_DIN0207_L6.3mm_D2.5mm_P7.62mm_Horizontal" (id 2) (at 125.222 158.75 90)
       (effects (font (size 1.27 1.27)) hide)
     )
@@
       (effects (font (size 1.27 1.27)) (justify left))
     )
-    (property "Value" "" (id 1) (at 260.35 91.4399 0)
-      (effects (font (size 1.27 1.27)) (justify left))
-    )
-    (property "Footprint" "" (id 2) (at 257.81 90.17 0)
+    (property "Value" "Servo_EXTRA" (id 1) (at 260.35 91.4399 0)
+      (effects (font (size 1.27 1.27)) (justify left))
+    )
+    (property "Footprint" "Connector_PinSocket_2.54mm:PinSocket_1x03_P2.54mm_Vertical" (id 2) (at 257.81 90.17 0)
       (effects (font (size 1.27 1.27)) hide)
     )
@@
     (in_bom yes) (on_board yes)
     (property "Reference" "J10" (id 0) (at 34.29 90.17 0))
-    (property "Value" "" (id 1) (at 29.21 82.55 0))
-    (property "Footprint" "" (id 2) (at 38.1 113.03 0)
+    (property "Value" "USB_C_Receptacle_USB2.0" (id 1) (at 29.21 82.55 0))
+    (property "Footprint" "Connector_USB:USB_C_Receptacle_GCT_USB4085" (id 2) (at 38.1 113.03 0)
       (effects (font (size 1.27 1.27)) hide)
     )
@@
       (effects (font (size 1.27 1.27)) (justify left))
     )
-    (property "Value" "" (id 1) (at 262.89 24.1299 0)
-      (effects (font (size 1.27 1.27)) (justify left))
-    )
-    (property "Footprint" "" (id 2) (at 260.35 21.59 0)
-      (effects (font (size 1.27 1.27)) hide)
-    )
+    (property "Value" "Motor_Driver_Left" (id 1) (at 262.89 24.1299 0)
+      (effects (font (size 1.27 1.27)) (justify left))
+    )
+    (property "Footprint" "Connector_PinSocket_2.54mm:PinSocket_1x04_P2.54mm_Vertical" (id 2) (at 260.35 21.59 0)
+      (effects (font (size 1.27 1.27)) hide)
+    )
